File: UV-Backlight-Prototype.kicad_pcb (KiCad board)
At the start: 2 copper layers, 86 parts, among them J1 Conn_02x08_Odd_Even

Commit message: Update UV-Backlight-Prototype.kicad_pcb
outline, mounting hole, connectors
Parts:
- LEDS 1: renamed from JP8
- LEDS 2: renamed from JP16
- LEDS 3: renamed from JP24
- moved H4 188.7 mm to (195.0, 135.0)
- moved H3 161.1 mm to (195.0, 45.0)
- moved J1 159.4 mm to (141.1, 133.8), turned to 90 degrees
- moved TP14 154.9 mm to (218.3, -11.9)
- moved TP11 154.9 mm to (209.6, -9.65)
- moved TP18 154.9 mm to (210.0, -14.0)
- moved TP3 154.9 mm to (213.9, -9.65)
- moved LEDS 3 152.0 mm to (156.2, 119.0), turned to 180 degrees
- moved TP15 144.8 mm to (203.0, -26.0)
- moved TP9 144.8 mm to (203.0, -21.6)
- moved LEDS 2 142.4 mm to (148.8, 119.0), turned to 180 degrees
- moved TH3 130.0 mm to (159.0, 22.0)
- moved LEDS 1 128.7 mm to (141.0, 119.0), turned to 180 degrees
- moved TP13 121.1 mm to (188.0, -33.0)
- moved H1 115.9 mm to (105.0, 135.0)
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Routing:
- added copper zone on B.Cu, net GND
- added copper zone on F.Cu, net GND
Other:
- board outline added: 100 x 100 mm
